File: rust/atmega168/schema/m168-lpd8806.kicad_pcb (KiCad board)
At the start: 4 copper layers, 75 x 51.8 mm, 4 parts, among them J1 Conn_01x06_Pin, U1 ATmega168P-20P

Commit message: Fahre mit Kicad fort
Changed lines of the file:
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@@
 	(net 0 "")
 	(net 1 "unconnected-(U1-PB1-Pad15)")
-	(net 2 "Net-(J1-Pin_2)")
+	(net 2 "Net-(J1-Reset)")
 	(net 3 "/Data")
 	(net 4 "/MISO")
@@
 			(layer "F.Fab")
 		)
+		(fp_text user "VCC"
+			(at 2.5 0 0)
+			(unlocked yes)
+			(layer "F.SilkS")
+			(effects
+				(font
+					(size 1 1)
+					(thickness 0.1)
+				)
+				(justify left bottom)
+			)
+		)
 		(fp_text user "${REFERENCE}"
 			(at 0 6.35 90)
@@
 			(remove_unused_layers no)
 			(net 8 "GND")
-			(pinfunction "Pin_1")
-			(pintype "passive")
+			(pinfunction "Gnd")
+			(pintype "power_in")
 		)
 		(pad "2" thru_hole circle
@@
 			(layers "*.Cu" "*.Mask")
 			(remove_unused_layers no)
-			(net 2 "Net-(J1-Pin_2)")
-			(pinfunction "Pin_2")
-			(pintype "passive")
+			(net 2 "Net-(J1-Reset)")
+			(pinfunction "Reset")
+			(pintype "input")
 		)
 		(pad "3" thru_hole circle
@@
 			(remove_unused_layers no)
 			(net 22 "+5V")
-			(pinfunction "Pin_6")
-			(pintype "passive")
+			(pinfunction "5V")
+			(pintype "power_in")
 		)
 		(embedded_fonts no)
@@
 			(remove_unused_layers no)
 			(roundrect_rratio 0.15625)
-			(net 2 "Net-(J1-Pin_2)")
+			(net 2 "Net-(J1-Reset)")
 			(pinfunction "~{RESET}/PC6")
 			(pintype "bidirectional")
